File: Enose_PCB.kicad_sch (KiCad schematic)
At the start: 0 parts

Commit message: Worked on the Schematic for the modem
Parts:
- added C? (x2): 1u, symbol Device:C
- added C?: 22u, symbol Device:C
- added C?: 0.1u, symbol Device:C
- added R? (x3): 10k, symbol Device:R
- added SW? (x2): SW_DPST_x2, symbol Switch:SW_DPST_x2
- added U?: ESP32-S3-WROOM-1, RF_Module:ESP32-S3-WROOM-1, symbol RF_Module:ESP32-S3-WROOM-1
Connections:
- new net: SW?.2 (B), U?.27 (IO0)
- new net +3V3: C?.1, C?.1, C?.2, R?.1, R?.1, R?.1, U?.2 (3V3)
- new net EN: C?.1, R?.2, R?.2, SW?.2 (B), U?.3 (EN)
- new net GND: C?.1, C?.2, C?.2, C?.2, SW?.1 (A), SW?.1 (A), U?.1 (GND), U?.40 (GND), U?.41 (GND)
- new net UART1_RXD: U?.37 (TXD0)
- new net UART1_TXD: R?.2, U?.36 (RXD0)
- new net USB_D+: U?.14 (IO20)
- new net USB_D-: U?.13 (IO19)
Other:
- added sheet Cellular Module (cellular.module.kicad_sch)
- added sheet Power (Power.kicad_sch)

Commit message: Added Power Components
Other:
- sheet Power renamed Power Components
Changed lines of the file:
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@@
 	)
 	(sheet
-		(at 114.3 165.1)
-		(size 44.45 19.05)
+		(at 95.25 158.75)
+		(size 63.5 31.75)
 		(exclude_from_sim no)
 		(in_bom yes)
@@
 		)
 		(fill
-			(color 0 0 0 0.0000)
+			(color 255 229 191 0.6000)
 		)
 		(property "Sheetname" "Cellular Module"
-			(at 114.3 164.3884 0)
+			(at 95.25 158.0384 0)
 			(effects
 				(font
 					(size 1.27 1.27)
+					(thickness 0.1588)
 				)
 				(justify left bottom)
@@
 		)
 		(property "Sheetfile" "cellular.module.kicad_sch"
-			(at 114.3 184.7346 0)
+			(at 95.25 191.0846 0)
 			(effects
 				(font
@@
 	)
 	(sheet
-		(at 36.83 163.83)
-		(size 44.45 20.32)
+		(at 21.59 158.75)
+		(size 63.5 31.75)
 		(exclude_from_sim no)
 		(in_bom yes)
@@
 		)
 		(fill
-			(color 0 0 0 0.0000)
+			(color 255 229 191 0.6000)
 		)
-		(property "Sheetname" "Power"
-			(at 36.83 163.1184 0)
+		(property "Sheetname" "Power Components"
+			(at 21.59 158.0384 0)
 			(effects
 				(font
@@
 		)
 		(property "Sheetfile" "Power.kicad_sch"
-			(at 36.83 184.7346 0)
+			(at 21.59 191.0846 0)
 			(effects
 				(font
