File: cellular.module.kicad_sch (KiCad schematic)
At the start: 42 parts

Commit message: Added Power Components
Parts:
- added J? (x2): U.FL-R-SMT_01_, U.FL-R-SMT_01_:HRS_U.FL-R-SMT_01_, symbol U.FL-R-SMT_01_:U.FL-R-SMT_01_
Connections:
- net GND: now also J?.1 (GND), J?.1 (GND), J?.2 (GND), J?.2 (GND)
- net GNSS_ANT: now reaches U?.53 (GNSS_ANT)
- net GNSS_ANT: now also J?.3 (SIG)
- net RF_ANT: now reaches U?.60 (RF_ANT)
- net RF_ANT: now also J?.3 (SIG)
- no-connect marks 20 -> 25
