File: Multi-emitter V2 Thesis/Multi-emitter V2 Thesis.kicad_sch (KiCad schematic)
At the start: 12 parts, among them J1 Emitter0 Input, J6 Emitter6 Input, Q1 NMOS

Commit message: redoing footprints
Parts:
- removed D1: DT1240A-08LP3810, Package_DFN_QFN:UDFN-9_1.0x3.8mm_P0.5mm, symbol Power_Protection:DT1240A-08LP3810
- added C2, C3, C4, C5, C6, C7, C8: 100n, Capacitor_SMD:C_0805_2012Metric_Pad1.18x1.45mm_HandSolder, symbol Device:C
- added J2, J3, J4, J5, J7, J8: Emitter Input, Connector_JST:JST_PH_S2B-PH-K_1x02_P2.00mm_Horizontal, symbol Connector:Screw_Terminal_01x02
- added L2, L3, L4, L5, L6, L7, L8: 220u, CDRH104FootprintLib:INDPM102100X400N, symbol Device:L
- added Q2, Q3, Q4, Q5, Q6, Q7, Q8: NMOS, Ventsi_Lib:Ventsi_SOT23, symbol Simulation_SPICE:NMOS
- added R2, R3, R4, R5, R6, R7, R8: 10k, Resistor_SMD:R_0805_2012Metric_Pad1.20x1.40mm_HandSolder, symbol Device:R
- C1: footprint Capacitor_THT:C_Disc_D5.0mm_W2.5mm_P5.00mm -> Capacitor_SMD:C_0805_2012Metric_Pad1.18x1.45mm_HandSolder
- J0: renamed from J?; footprint KiCad:XM3B1522112 -> XM3B_Lib:XM3B1522112
- J1: value Emitter0 Input -> Emitter Input; footprint TerminalBlock:TerminalBlock_bornier-2_P5.08mm -> Connector_JST:JST_PH_S2B-PH-K_1x02_P2.00mm_Horizontal
- J6: value Emitter6 Input -> Emitter Input; footprint TerminalBlock:TerminalBlock_bornier-2_P5.08mm -> Connector_JST:JST_PH_S2B-PH-K_1x02_P2.00mm_Horizontal
- L1: footprint Inductor_THT:L_Radial_D7.2mm_P3.00mm_Murata_1700 -> CDRH104FootprintLib:INDPM102100X400N
- Q1: footprint Package_DIP:Vishay_HVM-DIP-3_W7.62mm -> Ventsi_Lib:Ventsi_SOT23
- R1: footprint Resistor_THT:R_Axial_DIN0207_L6.3mm_D2.5mm_P10.16mm_Horizontal -> Resistor_SMD:R_0805_2012Metric_Pad1.20x1.40mm_HandSolder
Connections:
- net GND: now also J2.2 (Pin_2), J3.2 (Pin_2), J4.2 (Pin_2), J5.2 (Pin_2), J7.2 (Pin_2), J8.2 (Pin_2), Q2.3 (S), Q3.3 (S), Q4.3 (S), Q5.3 (S), Q6.3 (S), Q7.3 (S), Q8.3 (S), R2.2, R3.2, R4.2, R5.2, R6.2, R7.2, R8.2
- net PWM2: now also Q2.2 (G), R2.1
- net PWM3: now also Q3.2 (G), R3.1
- net PWM4: now also Q4.2 (G), R4.1
- net PWM5: now also Q5.2 (G), R5.1
- net PWM6: now also Q6.2 (G), R6.1
- net PWM7: now also Q7.2 (G)
- net PWM8: now also Q8.2 (G), R8.1
- net VCC: now also L2.1, L3.1, L4.1, L5.1, L6.1, L7.1, L8.1
- net at J6.1 (Pin_1): now also C7.2
- new net: C8.1, L5.2, Q5.1 (D)
- new net: C8.2, J5.1 (Pin_1)
- new net: C6.1, L7.2, Q7.1 (D)
- new net: C7.1, L6.2, Q6.1 (D)
- new net: C2.1, L2.2, Q2.1 (D)
- new net: C5.2, J8.1 (Pin_1)
- new net: C4.1, L4.2, Q4.1 (D)
- new net: C4.2, J4.1 (Pin_1)
- new net: C3.1, L3.2, Q3.1 (D)
- new net: C6.2, J7.1 (Pin_1)
- new net: C3.2, J3.1 (Pin_1)
- new net: C5.1, L8.2, Q8.1 (D)
- new net: C2.2, J2.1 (Pin_1)
Other:
- note added: "Dsub 15 connector with power, GND and PWM inputs"
- note added: "Emitter Drivers"
- note added: "Notes: 1. PWM inputs typical signal behaviour is either off state or 100-115 kHz 50% duty cycle square wave. 2. VCC should be between 13-16V. 3. Dangerous scenario if PWM inputs are too high/low frequencies."
- note added: "TODO: 2. Add LED indicator for power Disregarded circuit ideas: 1.complex emitter driver circuit (ideal sine wave for ideal driving) 2. BP filter on input to act as protection from too low or too high frequencies (it will distort the pwm signal which would aquire a shcmitt trigger to restore the vertical square wave edges which makes it more complex and costly) 3. Removed ESD protection on Dsub i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"
- note removed: "Amplifiers (Emitter Drivers)"
- note removed: "Connector + ESD protection"
- note removed: "Notes: 1.PWM inputs typical signal behaviour is either off state or 100-115 kHz. 2.VCC should be between 13-16V."
- note removed: "TODO: 1. Verify if the DT1240A-08LP3810Q is a good ESD IC 2. Add 2-pin JST connectors to match the emitter JST so they can easily be plugged in without havign to modify the wire ends. flyback diode on input filter not needed as currents are very low 3. Add a fuse to protect mosfet short circuit event (can happen if PWM inputs are either DC high or are driving at very high frequency) 4. Change som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"

Commit message: PCB layout done on emitter PCB - ready to order
Parts:
- added D2: LED, LED_THT:LED_D5.0mm, symbol Device:LED
- added R9: 1k, Resistor_SMD:R_0805_2012Metric_Pad1.20x1.40mm_HandSolder, symbol Device:R
- renumbered C8 to C5, C7 to C6, C6 to C7, C5 to C8
Connections:
- net GND: now also D2.1 (K)
- net PWM7: now also R7.1
- net VCC: now also R9.1
- new net: D2.2 (A), R9.2
Other:
- note added: "Discarded circuit ideas: 1. Complex emitter driver circuit (ideal sine wave for ideal driving) 2. BP filter on input to act as protection from too low or too high frequencies (it will distort the pwm signal which would aquire a shcmitt trigger to restore the vertical square wave edges which makes it more complex and costly) 3. Removed ESD protection on Dsub input since mosfet gates already have i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"
- note added: "Notes: 1. PWM inputs typical signal behaviour is either off state or 100-115 kHz 50% duty cycle square wave. 2. VCC should be between 13-16V. 3. Dangerous scenario if PWM inputs are too high/low frequencies. 4. N-mos gates include ESD protection."
- note added: "Power Indicator Diode"
- note removed: "Notes: 1. PWM inputs typical signal behaviour is either off state or 100-115 kHz 50% duty cycle square wave. 2. VCC should be between 13-16V. 3. Dangerous scenario if PWM inputs are too high/low frequencies."
- note removed: "TODO: 2. Add LED indicator for power Disregarded circuit ideas: 1.complex emitter driver circuit (ideal sine wave for ideal driving) 2. BP filter on input to act as protection from too low or too high frequencies (it will distort the pwm signal which would aquire a shcmitt trigger to restore the vertical square wave edges which makes it more complex and costly) 3. Removed ESD protection on Dsub i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"
- moved on the sheet: H1, H2, H3, H4
